File: PCB/binaryclock.sch (KiCad schematic (older format))
At the start: 13 parts, among them IC1 ATMEGA328P-P

Commit message: Components placed on PCB and connections made in drawing mode.
Parts:
- added HLS1, HLS2, HLS3, HLS4, HLS5, HLS6, HMS1, HMS2, HMS3, MMS1, MMS2, MMS3: LED, LEDs:LED-3MM, symbol LED
- added R10, R11, R12, R13, R14, R15, R16, R17, R18, R7, R8, R9: 220, Resistors_ThroughHole:Resistor_Horizontal_RM10mm, symbol R
- added SW1, SW2: SW_PUSH, Buttons_Switches_SMD:SW_SPST_EVQP2, symbol SW_PUSH
- R6: footprint Resistors_ThroughHole:Resistor_Ceramic_Horizontal_L19mm-W8mm-H8mm-p25mm -> Resistors_ThroughHole:Resistor_Horizontal_RM10mm
- renumbered D1 to MLS1, D2 to MLS2, D3 to MLS3, D4 to MLS4, D5 to MLS5, D6 to MLS6
Connections:
- net +3V3 is gone; now on net +5V: IC1.7 (VCC)
- net GND: now also HLS1.1 (K), HLS2.1 (K), HLS3.1 (K), HLS4.1 (K), HLS5.1 (K), HLS6.1 (K), HMS1.1 (K), HMS2.1 (K), HMS3.1 (K), MMS1.1 (K), MMS2.1 (K), MMS3.1 (K), SW1.2, SW2.2
- net minute_leastsig_3: now also IC1.6 ((PCINT20/XCK/T0)PD4); no longer IC1.4 ((PCINT18/INT0)PD2)
- net minute_leastsig_4: now also IC1.11 ((PCINT21/OC0B/T1)PD5); no longer IC1.5 ((PCINT19/OC2B/INT1)PD3)
- net minute_leastsig_5: now also IC1.12 ((PCINT22/OC0A/AIN0)PD6); no longer IC1.6 ((PCINT20/XCK/T0)PD4)
- net minute_leastsig_6: now also IC1.13 ((PCINT23/AIN1)PD7); no longer IC1.11 ((PCINT21/OC0B/T1)PD5)
- net +5V: now reaches IC1.1 ((PCINT14/~RESET~)PC6)
- net hour_leastsig_3: now reaches IC1.10 ((PCINT7/XTAL2/TOSC2)PB7)
- net hour_leastsig_3: now also R12.2
- net hour_mostsig_1: now reaches IC1.17 ((PCINT3/OC2A/MOSI)PB3)
- net hour_mostsig_1: now also R16.2, R17.2, R18.2
- net hour_mostsig_2: now reaches IC1.18 ((PCINT4/MISO)PB4)
- net hour_leastsig_1: now reaches IC1.19 ((PCINT5/SCK)PB5)
- net hour_leastsig_1: now also R10.2
- net hour_leastsig_4: now reaches IC1.23 ((PCINT8/ADC0)PC0)
- net hour_leastsig_4: now also R13.2
- net hour_leastsig_5: now reaches IC1.24 ((PCINT9/ADC1)PC1)
- net hour_leastsig_5: now also R14.2
- net hour_leastsig_6: now reaches IC1.25 ((PCINT10/ADC2)PC2)
- net minute_mostsig_1: now reaches IC1.26 ((PCINT11/ADC3)PC3)
- net minute_mostsig_1: now also R7.2
- net minute_mostsig_2: now reaches IC1.27 ((PCINT12/SDA/ADC4)PC4)
- net minute_mostsig_2: now also R8.2
- net minute_mostsig_3: now reaches IC1.28 ((PCINT13/SCL/ADC5)PC5)
- net minute_mostsig_3: now also R9.2
- net hour_leastsig_2: now reaches IC1.9 ((PCINT6/XTAL1/TOSC1)PB6)
- net hour_leastsig_2: now also R11.2, R15.2
- new net: MMS1.2 (A), R7.1
- new net: MMS2.2 (A), R8.1
- new net: MMS3.2 (A), R9.1
- new net: HLS1.2 (A), R10.1
- new net: HLS2.2 (A), R11.1
- new net: HLS3.2 (A), R12.1
- new net: HLS4.2 (A), R13.1
- new net: HLS5.2 (A), R14.1
- new net: HLS6.2 (A), R15.1
- new net: HMS1.2 (A), R16.1
- new net: HMS2.2 (A), R17.1
- new net: HMS3.2 (A), R18.1
- new net add_hour: IC1.5 ((PCINT19/OC2B/INT1)PD3), SW2.1
- new net add_minute: IC1.4 ((PCINT18/INT0)PD2), SW1.1
- no-connect marks 2 -> 5
